File: KiCad/SignalSnagger/SignalSnagger.kicad_sch (KiCad schematic)
At the start: 57 parts, among them J101 Left, J103 Right, Q101 MMBT2222A, Q102 MMBT2222A, Q103 MMBT2222A, SW101 Sense, T101 Transformer_1P_SS, U101 74HC74, U103 LT6231

Commit message: Schematic Update
Parts:
- added J108: 36-5005-ND, symbol Connector_Generic:Conn_01x01
- AE102: value (none) -> Antenna_80m_DF
- C103: value (none) -> 8.5-100pF
- C104: value (none) -> 51pF
- J102: value (none) -> Left
- J104: value (none) -> Right
- J105: value (none) -> 36-5005-ND
- J106, J107: value (none) -> 36-5006-ND
- RV101: value (none) -> 10k 10T
- RV102: value (none) -> 50k
- U102: value (none) -> QS3253QG8
Connections:
- net at AE101.1 (A), C101.1: now also J108.1 (Pin_1)
Other:
- note added: "Nominal 14.2 MHz"
Changed lines of the file:
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@@
     (title "SignalSnagger")
     (date "2023-11-05")
-    (rev "0.7")
+    (rev "0.8")
   )
   (junction (at 190.5 113.03) (diameter 0) (color 0 0 0 0)
@@
   )
   (junction (at 218.44 92.71) (diameter 0) (color 0 0 0 0)
+  )
+  (junction (at 21.59 52.07) (diameter 0) (color 0 0 0 0)
   )
   (junction (at 115.57 119.38) (diameter 0) (color 0 0 0 0)
@@
     (stroke (width 0) (type default) (color 0 0 0 0))
   )
-  (wire (pts (xy 21.59 111.76) (xy 21.59 33.02))
+  (wire (pts (xy 21.59 111.76) (xy 21.59 52.07))
     (stroke (width 0) (type default) (color 0 0 0 0))
   )
@@
   )
   (wire (pts (xy 218.44 109.22) (xy 218.44 107.95))
+    (stroke (width 0) (type default) (color 0 0 0 0))
+  )
+  (wire (pts (xy 21.59 52.07) (xy 21.59 33.02))
     (stroke (width 0) (type default) (color 0 0 0 0))
   )
@@
   )
   (text "Secondary" (at 152.4 101.6 0)
+    (effects (font (size 1.27 1.27)) (justify left bottom))
+  )
+  (text "Nominal 14.2 MHz" (at 106.68 39.37 0)
     (effects (font (size 1.27 1.27)) (justify left bottom))
   )
@@
       (effects (font (size 1.27 1.27)) (justify left))
     )
-    (property "Value" "" (id 1) (at 100.33 63.5 0)
+    (property "Value" "36-5005-ND" (id 1) (at 100.33 63.5 0)
       (effects (font (size 1.27 1.27)) (justify left))
     )
@@
       (effects (font (size 1.27 1.27)) (justify right))
     )
-    (property "Value" "" (id 1) (at 126.111 98.2222 0)
+    (property "Value" "50k" (id 1) (at 126.111 98.2222 0)
       (effects (font (size 1.27 1.27)) (justify right))
     )
@@
       (effects (font (size 1.27 1.27)) (justify left))
     )
-    (property "Value" "" (id 1) (at 205.74 45.72 0)
+    (property "Value" "QS3253QG8" (id 1) (at 205.74 45.72 0)
       (effects (font (size 1.27 1.27)) (justify left))
     )
@@
     (in_bom yes) (on_board yes) (fields_autoplaced)
     (property "Reference" "J104" (id 0) (at 69.85 68.6902 0))
-    (property "Value" "" (id 1) (at 69.85 71.2271 0))
+    (property "Value" "Right" (id 1) (at 69.85 71.2271 0))
     (property "Footprint" "" (id 2) (at 68.58 76.2 0)
       (effects (font (size 1.27 1.27)) hide)
@@
     (in_bom yes) (on_board yes)
     (property "Reference" "C103" (id 0) (at 90.17 73.66 90))
-    (property "Value" "" (id 1) (at 91.44 76.2 90))
+    (property "Value" "8.5-100pF" (id 1) (at 91.44 76.2 90))
     (property "Footprint" "" (id 2) (at 90.17 78.74 0)
       (effects (font (size 1.27 1.27)) hide)
@@
     (in_bom yes) (on_board yes)
     (property "Reference" "C104" (id 0) (at 90.17 83.82 90))
-    (property "Value" "" (id 1) (at 90.17 88.9 90))
+    (property "Value" "51pF" (id 1) (at 90.17 88.9 90))
     (property "Footprint" "" (id 2) (at 90.17 86.36 0)
       (effects (font (size 1.27 1.27)) hide)
@@
       (effects (font (size 1.27 1.27)) (justify left))
     )
-    (property "Value" "" (id 1) (at 87.63 55.88 0)
+    (property "Value" "36-5006-ND" (id 1) (at 87.63 55.88 0)
       (effects (font (size 1.27 1.27)) (justify left))
     )
@@
     (in_bom yes) (on_board yes) (fields_autoplaced)
     (property "Reference" "J102" (id 0) (at 45.72 68.6902 0))
-    (property "Value" "" (id 1) (at 45.72 71.2271 0))
+    (property "Value" "Left" (id 1) (at 45.72 71.2271 0))
     (property "Footprint" "" (id 2) (at 44.45 76.2 0)
       (effects (font (size 1.27 1.27)) hide)
@@
     (in_bom yes) (on_board yes)
     (property "Reference" "RV101" (id 0) (at 33.02 116.84 90))
-    (property "Value" "" (id 1) (at 36.83 124.46 90))
+    (property "Value" "10k 10T" (id 1) (at 36.83 124.46 90))
     (property "Footprint" "" (id 2) (at 34.29 124.46 0)
       (effects (font (size 1.27 1.27)) hide)
@@
     (in_bom yes) (on_board yes)
     (property "Reference" "AE102" (id 0) (at 77.47 19.2622 0))
-    (property "Value" "" (id 1) (at 77.47 21.7991 0))
+    (property "Value" "Antenna_80m_DF" (id 1) (at 77.47 21.7991 0))
     (property "Footprint" "" (id 2) (at 78.74 27.94 0)
       (effects (font (size 1.27 1.27)) hide)
@@
     (pin "2")
   )
+  (symbol (lib_id "Connector_Generic:Conn_01x01") (at 26.67 52.07 0) (unit 1)
+    (in_bom yes) (on_board yes)
+    (property "Reference" "J108" (id 0) (at 28.702 51.2353 0)
+      (effects (font (size 1.27 1.27)) (justify left))
+    )
+    (property "Value" "36-5005-ND" (id 1) (at 19.05 55.88 0)
+      (effects (font (size 1.27 1.27)) (justify left))
+    )
+    (property "Footprint" "" (id 2) (at 26.67 52.07 0)
+      (effects (font (size 1.27 1.27)) hide)
+    )
+    (property "Datasheet" "~" (id 3) (at 26.67 52.07 0)
+      (effects (font (size 1.27 1.27)) hide)
+    )
+    (pin "1")
+  )
   (symbol (lib_id "power:GND") (at 90.17 52.07 0) (unit 1)
     (in_bom yes) (on_board yes) (fields_autoplaced)
@@
       (effects (font (size 1.27 1.27)) (justify left))
     )
-    (property "Value" "" (id 1) (at 101.6 55.88 0)
+    (property "Value" "36-5006-ND" (id 1) (at 101.6 55.88 0)
       (effects (font (size 1.27 1.27)) (justify left))
     )
@@
       (reference "J107") (unit 1) (value "36-5006-ND") (footprint "")
     )
+    (path "/d7d31544-a2bf-4ba0-8307-8924e326bbdf"
+      (reference "J108") (unit 1) (value "36-5005-ND") (footprint "")
+    )
     (path "/b7e6c0d8-791a-469a-85d5-f8e886443224/87efc960-fc20-4947-aae8-fb6b9c89ea87"
