File: KiCad/SignalSnagger/SignalSnagger.kicad_sch (KiCad schematic)
At the start: 81 parts, among them J101 Left, J103 Right, J105 36-5005-ND, J106 36-5006-ND, J107 36-5006-ND, J108 36-5005-ND, J909 36-5006-ND, J910 36-5006-ND, Q101 MMBT2222A, Q102 MMBT2222A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

Commit message: Schematic PDF File
Updated date on schematic and printed an updated PDF schematic. No changes made to design.
Parts:
- J102, J104: value (none) -> 69830-008LF; footprint (none) -> Connector_Amphenol:69830-008LF
Changed lines of the file:
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@@
   (title_block
     (title "SignalSnagger")
-    (date "2024-04-13")
+    (date "2024-05-03")
     (rev "0.317")
   )
@@
     (in_bom yes) (on_board yes) (fields_autoplaced)
     (property "Reference" "J104" (id 0) (at 69.85 87.7372 0))
-    (property "Value" "" (id 1) (at 69.85 87.7371 0)
-      (effects (font (size 1.27 1.27)) hide)
-    )
-    (property "Footprint" "" (id 2) (at 68.58 92.71 0)
+    (property "Value" "69830-008LF" (id 1) (at 69.85 87.7371 0)
+      (effects (font (size 1.27 1.27)) hide)
+    )
+    (property "Footprint" "Connector_Amphenol:69830-008LF" (id 2) (at 68.58 92.71 0)
       (effects (font (size 1.27 1.27)) hide)
     )
@@
     (in_bom yes) (on_board yes) (fields_autoplaced)
     (property "Reference" "J102" (id 0) (at 45.72 87.7372 0))
-    (property "Value" "" (id 1) (at 45.72 87.7371 0)
-      (effects (font (size 1.27 1.27)) hide)
-    )
-    (property "Footprint" "" (id 2) (at 44.45 92.71 0)
-      (effects (font (size 1.27 1.27)) hide)
-    )
+    (property "Value" "69830-008LF" (id 1) (at 45.72 87.7371 0)
+      (effects (font (size 1.27 1.27)) hide)
+    )
+    (property "Footprint" "Connector_Amphenol:69830-008LF" (id 2) (at 44.45 92.71 0)
+      (effects (font (size 1.27 1.27)) hide)
+    )
