File: KiCad/SignalSnagger/audio.kicad_sch (KiCad schematic)
At the start: 33 parts, among them J301 AudioJack4, U301 LM386, U302 LT6231

Commit message: Schematic Updates
Rev 0.18
Parts:
- added R314: 49.9k, symbol Device:R_US
- added R315: 10k, symbol Device:R_US
- C308: value 220uF -> (none)
Connections:
- net GND: now also R315.2
- net I OUT: now also R314.1
- net Q OUT: now also R310.1
- net at C309.1, C311.1, C313.1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: no longer R310.1
- net Audio renamed Audio Q
- new net Audio I: R314.2, R315.1
- no-connect marks 2 -> 1
Other:
- moved on the sheet: R310, R311
Changed lines of the file:
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@@
   (title_block
     (title "SignalSnagger")
-    (date "2023-12-10")
-    (rev "0.16")
-  )
-  (junction (at 120.65 130.81) (diameter 0) (color 0 0 0 0)
+    (date "2023-12-19")
+    (rev "0.18")
+  )
+  (junction (at 66.04 128.27) (diameter 0) (color 0 0 0 0)
   )
   (junction (at 99.06 116.84) (diameter 0) (color 0 0 0 0)
@@
   (junction (at 190.5 49.53) (diameter 0) (color 0 0 0 0)
   )
+  (junction (at 72.39 58.42) (diameter 0) (color 0 0 0 0)
+  )
   (junction (at 129.54 119.38) (diameter 0) (color 0 0 0 0)
   )
@@
   (junction (at 184.15 72.39) (diameter 0) (color 0 0 0 0)
   )
+  (junction (at 66.04 116.84) (diameter 0) (color 0 0 0 0)
+  )
   (junction (at 180.34 59.69) (diameter 0) (color 0 0 0 0)
   )
   (no_connect (at 217.17 59.69))
-  (no_connect (at 80.01 57.15))
   (wire (pts (xy 182.88 119.38) (xy 185.42 119.38))
     (stroke (width 0) (type default) (color 0 0 0 0))
@@
     (stroke (width 0) (type default) (color 0 0 0 0))
   )
+  (wire (pts (xy 66.04 116.84) (xy 74.93 116.84))
+    (stroke (width 0) (type default) (color 0 0 0 0))
+  )
   (wire (pts (xy 182.88 120.65) (xy 182.88 119.38))
     (stroke (width 0) (type default) (color 0 0 0 0))
   )
+  (wire (pts (xy 60.96 50.8) (xy 72.39 50.8))
+    (stroke (width 0) (type default) (color 0 0 0 0))
+  )
   (wire (pts (xy 158.75 50.8) (xy 158.75 55.88))
     (stroke (width 0) (type default) (color 0 0 0 0))
@@
     (stroke (width 0) (type default) (color 0 0 0 0))
   )
+  (wire (pts (xy 72.39 58.42) (xy 76.2 58.42))
+    (stroke (width 0) (type default) (color 0 0 0 0))
+  )
   (wire (pts (xy 147.32 50.8) (xy 148.59 50.8))
     (stroke (width 0) (type default) (color 0 0 0 0))
@@
     (stroke (width 0) (type default) (color 0 0 0 0))
   )
+  (wire (pts (xy 60.96 116.84) (xy 66.04 116.84))
+    (stroke (width 0) (type default) (color 0 0 0 0))
+  )
   (wire (pts (xy 190.5 43.18) (xy 191.77 43.18))
     (stroke (width 0) (type default) (color 0 0 0 0))
@@
     (stroke (width 0) (type default) (color 0 0 0 0))
   )
-  (wire (pts (xy 74.93 57.15) (xy 80.01 57.15))
-    (stroke (width 0) (type default) (color 0 0 0 0))
-  )
   (wire (pts (xy 198.12 77.47) (xy 198.12 69.85))
     (stroke (width 0) (type default) (color 0 0 0 0))
@@
     (stroke (width 0) (type default) (color 0 0 0 0))
   )
-  (wire (pts (xy 120.65 119.38) (xy 120.65 123.19))
+  (wire (pts (xy 66.04 116.84) (xy 66.04 120.65))
     (stroke (width 0) (type default) (color 0 0 0 0))
   )
@@
     (stroke (width 0) (type default) (color 0 0 0 0))
   )
-  (wire (pts (xy 120.65 130.81) (xy 124.46 130.81))
+  (wire (pts (xy 66.04 128.27) (xy 69.85 128.27))
     (stroke (width 0) (type default) (color 0 0 0 0))
   )
@@
     (stroke (width 0) (type default) (color 0 0 0 0))
   )
+  (wire (pts (xy 72.39 59.69) (xy 72.39 58.42))
+    (stroke (width 0) (type default) (color 0 0 0 0))
+  )
   (wire (pts (xy 85.09 116.84) (xy 85.09 121.92))
     (stroke (width 0) (type default) (color 0 0 0 0))
@@
     (stroke (width 0) (type default) (color 0 0 0 0))
   )
-  (wire (pts (xy 120.65 132.08) (xy 120.65 130.81))
+  (wire (pts (xy 66.04 129.54) (xy 66.04 128.27))
     (stroke (width 0) (type default) (color 0 0 0 0))
   )
@@
     )
   )
-  (global_label "Audio" (shape output) (at 124.46 130.81 0) (fields_autoplaced)
+  (global_label "Audio Q" (shape output) (at 69.85 128.27 0) (fields_autoplaced)
     (effects (font (size 1 1)) (justify left))
-    (property "Intersheet References" "${INTERSHEET_REFS}" (id 0) (at 130.4076 130.7475 0)
+    (property "Intersheet References" "${INTERSHEET_REFS}" (id 0) (at 77.6071 128.2075 0)
       (effects (font (size 1 1)) (justify left) hide)
     )
@@
     )
   )
-  (global_label "Q OUT" (shape input) (at 74.93 116.84 180) (fields_autoplaced)
+  (global_label "Q OUT" (shape input) (at 60.96 116.84 180) (fields_autoplaced)
     (effects (font (size 1 1)) (justify right))
-    (property "Intersheet References" "${INTERSHEET_REFS}" (id 0) (at 68.3633 116.7775 0)
+    (property "Intersheet References" "${INTERSHEET_REFS}" (id 0) (at 54.3933 116.7775 0)
       (effects (font (size 1 1)) (justify right) hide)
     )
@@
     )
   )
-  (global_label "I OUT" (shape input) (at 74.93 57.15 180) (fields_autoplaced)
+  (global_label "I OUT" (shape input) (at 60.96 50.8 180) (fields_autoplaced)
     (effects (font (size 1 1)) (justify right))
-    (property "Intersheet References" "${INTERSHEET_REFS}" (id 0) (at 68.9348 57.0875 0)
+    (property "Intersheet References" "${INTERSHEET_REFS}" (id 0) (at 54.9648 50.7375 0)
       (effects (font (size 1 1)) (justify right) hide)
+    )
+  )
+  (global_label "Audio I" (shape output) (at 76.2 58.42 0) (fields_autoplaced)
+    (effects (font (size 1 1)) (justify left))
+    (property "Intersheet References" "${INTERSHEET_REFS}" (id 0) (at 83.3857 58.3575 0)
+      (effects (font (size 1 1)) (justify left) hide)
     )
   )
@@
     (pin "S")
     (pin "T")
+  )
+  (symbol (lib_id "Device:R_US") (at 72.39 54.61 0) (unit 1)
+    (in_bom yes) (on_board yes)
+    (property "Reference" "R314" (id 0) (at 69.85 54.61 90))
+    (property "Value" "49.9k" (id 1) (at 74.4419 54.61 90))
+    (property "Footprint" "" (id 2) (at 73.406 54.864 90)
+      (effects (font (size 1.27 1.27)) hide)
+    )
+    (property "Datasheet" "~" (id 3) (at 72.39 54.61 0)
+      (effects (font (size 1.27 1.27)) hide)
+    )
+    (pin "1")
+    (pin "2")
   )
   (symbol (lib_id "Device:C_Small") (at 111.76 110.49 90) (unit 1)
@@
     (pin "2")
   )
-  (symbol (lib_id "power:GND") (at 120.65 139.7 0) (unit 1)
-    (in_bom yes) (on_board yes) (fields_autoplaced)
-    (property "Reference" "#PWR0319" (id 0) (at 120.65 146.05 0)
-      (effects (font (size 1.27 1.27)) hide)
-    )
-    (property "Value" "GND" (id 1) (at 120.65 144.1434 0))
-    (property "Footprint" "" (id 2) (at 120.65 139.7 0)
-      (effects (font (size 1.27 1.27)) hide)
-    )
-    (property "Datasheet" "" (id 3) (at 120.65 139.7 0)
+  (symbol (lib_id "power:GND") (at 66.04 137.16 0) (unit 1)
+    (in_bom yes) (on_board yes) (fields_autoplaced)
+    (property "Reference" "#PWR0319" (id 0) (at 66.04 143.51 0)
+      (effects (font (size 1.27 1.27)) hide)
+    )
+    (property "Value" "GND" (id 1) (at 66.04 141.6034 0))
+    (property "Footprint" "" (id 2) (at 66.04 137.16 0)
+      (effects (font (size 1.27 1.27)) hide)
+    )
+    (property "Datasheet" "" (id 3) (at 66.04 137.16 0)
       (effects (font (size 1.27 1.27)) hide)
     )
@@
     (pin "2")
   )
-  (symbol (lib_id "Device:R_US") (at 120.65 127 0) (unit 1)
-    (in_bom yes) (on_board yes)
-    (property "Reference" "R310" (id 0) (at 118.11 127 90))
-    (property "Value" "49.9k" (id 1) (at 122.7019 127 90))
-    (property "Footprint" "" (id 2) (at 121.666 127.254 90)
-      (effects (font (size 1.27 1.27)) hide)
-    )
-    (property "Datasheet" "~" (id 3) (at 120.65 127 0)
-      (effects (font (size 1.27 1.27)) hide)
-    )
-    (pin "1")
-    (pin "2")
-  )
-  (symbol (lib_id "Device:R_US") (at 120.65 135.89 0) (unit 1)
-    (in_bom yes) (on_board yes)
-    (property "Reference" "R311" (id 0) (at 118.11 135.89 90))
-    (property "Value" "10k" (id 1) (at 122.7019 135.89 90))
-    (property "Footprint" "" (id 2) (at 121.666 136.144 90)
-      (effects (font (size 1.27 1.27)) hide)
-    )
-    (property "Datasheet" "~" (id 3) (at 120.65 135.89 0)
+  (symbol (lib_id "Device:R_US") (at 66.04 124.46 0) (unit 1)
+    (in_bom yes) (on_board yes)
+    (property "Reference" "R310" (id 0) (at 63.5 124.46 90))
+    (property "Value" "49.9k" (id 1) (at 68.0919 124.46 90))
+    (property "Footprint" "" (id 2) (at 67.056 124.714 90)
+      (effects (font (size 1.27 1.27)) hide)
+    )
+    (property "Datasheet" "~" (id 3) (at 66.04 124.46 0)
+      (effects (font (size 1.27 1.27)) hide)
+    )
+    (pin "1")
+    (pin "2")
+  )
+  (symbol (lib_id "Device:R_US") (at 66.04 133.35 0) (unit 1)
+    (in_bom yes) (on_board yes)
+    (property "Reference" "R311" (id 0) (at 63.5 133.35 90))
+    (property "Value" "10k" (id 1) (at 68.0919 133.35 90))
+    (property "Footprint" "" (id 2) (at 67.056 133.604 90)
+      (effects (font (size 1.27 1.27)) hide)
+    )
+    (property "Datasheet" "~" (id 3) (at 66.04 133.35 0)
       (effects (font (size 1.27 1.27)) hide)
     )
@@
   (symbol (lib_id "Device:C_Small") (at 208.28 62.23 270) (unit 1)
     (in_bom yes) (on_board yes)
-    (property "Reference" "C308" (id 0) (at 209.55 58.42 90)
-      (effects (font (size 1.27 1.27)) (justify right))
-    )
-    (property "Value" "220uF" (id 1) (at 212.09 64.77 90)
+    (property "Reference" "C308" (id 0) (at 210.82 59.69 90)
+      (effects (font (size 1.27 1.27)) (justify right))
+    )
+    (property "Value" "" (id 1) (at 212.09 64.77 90)
       (effects (font (size 1.27 1.27)) (justify right))
     )
@@
     )
     (property "Datasheet" "~" (id 3) (at 196.85 53.34 0)
+      (effects (font (size 1.27 1.27)) hide)
+    )
+    (pin "1")
+    (pin "2")
+  )
+  (symbol (lib_id "Device:R_US") (at 72.39 63.5 0) (unit 1)
+    (in_bom yes) (on_board yes)
+    (property "Reference" "R315" (id 0) (at 69.85 63.5 90))
+    (property "Value" "10k" (id 1) (at 74.4419 63.5 90))
+    (property "Footprint" "" (id 2) (at 73.406 63.754 90)
+      (effects (font (size 1.27 1.27)) hide)
+    )
+    (property "Datasheet" "~" (id 3) (at 72.39 63.5 0)
       (effects (font (size 1.27 1.27)) hide)
     )
@@
       (effects (font (size 1.27 1.27)) hide)
     )
+    (pin "1")
+  )
+  (symbol (lib_id "power:GND") (at 72.39 67.31 0) (unit 1)
+    (in_bom yes) (on_board yes) (fields_autoplaced)
+    (property "Reference" "#PWR0152" (id 0) (at 72.39 73.66 0)
+      (effects (font (size 1.27 1.27)) hide)
+    )
+    (property "Value" "GND" (id 1) (at 72.39 71.7534 0))
+    (property "Footprint" "" (id 2) (at 72.39 67.31 0)
+      (effects (font (size 1.27 1.27)) hide)
+    )
+    (property "Datasheet" "" (id 3) (at 72.39 67.31 0)
+      (effects (font (size 1.27 1.27)) hide)
+    )

Commit message: Schematic Tweaks
Connections:
- net +9V renamed +VSW
Changed lines of the file:
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@@
     (pin "2")
-  )
-  (symbol (lib_id "power:+9V") (at 190.5 31.75 0) (unit 1)
-    (in_bom yes) (on_board yes)
-    (property "Reference" "#PWR0304" (id 0) (at 190.5 35.56 0)
-      (effects (font (size 1.27 1.27)) hide)
-    )
-    (property "Value" "+9V" (id 1) (at 190.5 27.94 0))
-    (property "Footprint" "" (id 2) (at 190.5 31.75 0)
-      (effects (font (size 1.27 1.27)) hide)
-    )
-    (property "Datasheet" "" (id 3) (at 190.5 31.75 0)
-      (effects (font (size 1.27 1.27)) hide)
-    )
-    (pin "1")
   )
   (symbol (lib_id "power:GND") (at 184.15 72.39 0) (unit 1)
@@
     (pin "2")
   )
+  (symbol (lib_id "power:+VSW") (at 190.5 31.75 0) (unit 1)
+    (in_bom yes) (on_board yes)
+    (property "Reference" "#PWR0153" (id 0) (at 190.5 35.56 0)
+      (effects (font (size 1.27 1.27)) hide)
+    )
+    (property "Value" "+VSW" (id 1) (at 187.96 27.94 0))
+    (property "Footprint" "" (id 2) (at 190.5 31.75 0)
+      (effects (font (size 1.27 1.27)) hide)
+    )
+    (property "Datasheet" "" (id 3) (at 190.5 31.75 0)
+      (effects (font (size 1.27 1.27)) hide)
+    )
+    (pin "1")
+  )
   (symbol (lib_id "Device:R_US") (at 66.04 133.35 0) (unit 1)

Commit message: Schematic Updates
First cut at prototype design
Parts:
- C308: value (none) -> 20uF
Changed lines of the file:
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@@
     (title "SignalSnagger")
     (date "2023-12-19")
-    (rev "0.18")
+    (rev "0.20")
   )
   (junction (at 66.04 128.27) (diameter 0) (color 0 0 0 0)
@@
       (effects (font (size 1.27 1.27)) (justify right))
     )
-    (property "Value" "" (id 1) (at 212.09 64.77 90)
-      (effects (font (size 1.27 1.27)) (justify right))
-    )
+    (property "Value" "20uF" (id 1) (at 212.09 64.77 90)
+      (effects (font (size 1.27 1.27)) (justify right))
+    )

Commit message: Ver 0.22
o Schematic updates
Parts:
- added R316: (no value), symbol Device:R_US
Connections:
- net GND: now also R316.2
- net at U301.8 (GAIN): no longer C305.1
- net ASSI renamed ASSI_NEAR
- new net: C305.1, R316.1
Other:
- moved on the sheet: C305
Changed lines of the file:
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@@
   (title_block
     (title "SignalSnagger")
-    (date "2023-12-19")
-    (rev "0.21")
+    (date "2024-02-01")
+    (rev "0.22")
   )
   (junction (at 66.04 128.27) (diameter 0) (color 0 0 0 0)
@@
     (stroke (width 0) (type default) (color 0 0 0 0))
   )
-  (wire (pts (xy 193.04 69.85) (xy 193.04 77.47))
+  (wire (pts (xy 193.04 69.85) (xy 193.04 72.39))
     (stroke (width 0) (type default) (color 0 0 0 0))
   )
@@
     (stroke (width 0) (type default) (color 0 0 0 0))
   )
-  (wire (pts (xy 198.12 77.47) (xy 198.12 69.85))
-    (stroke (width 0) (type default) (color 0 0 0 0))
-  )
   (wire (pts (xy 180.34 59.69) (xy 185.42 59.69))
     (stroke (width 0) (type default) (color 0 0 0 0))
@@
   )
   (wire (pts (xy 180.34 68.58) (xy 180.34 72.39))
-    (stroke (width 0) (type default) (color 0 0 0 0))
-  )
-  (wire (pts (xy 198.12 69.85) (xy 195.58 69.85))
     (stroke (width 0) (type default) (color 0 0 0 0))
   )
@@
     )
   )
-  (global_label "ASSI" (shape output) (at 185.42 119.38 0) (fields_autoplaced)
+  (global_label "ASSI_NEAR" (shape output) (at 185.42 119.38 0) (fields_autoplaced)
     (effects (font (size 1 1)) (justify left))
-    (property "Intersheet References" "${INTERSHEET_REFS}" (id 0) (at 190.5581 119.3175 0)
+    (property "Intersheet References" "${INTERSHEET_REFS}" (id 0) (at 195.1295 119.3175 0)
       (effects (font (size 1 1)) (justify left) hide)
     )
@@
     (pin "1")
   )
+  (symbol (lib_id "Device:R_US") (at 193.04 81.28 0) (unit 1)
+    (in_bom yes) (on_board yes) (fields_autoplaced)
+    (property "Reference" "R316" (id 0) (at 194.691 80.4453 0)
+      (effects (font (size 1.27 1.27)) (justify left))
+    )
+    (property "Value" "" (id 1) (at 194.691 82.9822 0)
+      (effects (font (size 1.27 1.27)) (justify left))
+    )
+    (property "Footprint" "" (id 2) (at 194.056 81.534 90)
+      (effects (font (size 1.27 1.27)) hide)
+    )
+    (property "Datasheet" "~" (id 3) (at 193.04 81.28 0)
+      (effects (font (size 1.27 1.27)) hide)
+    )
+    (pin "1")
+    (pin "2")
+  )
   (symbol (lib_id "Device:R_US") (at 78.74 116.84 90) (unit 1)
     (in_bom yes) (on_board yes)
@@
     (pin "1")
   )
-  (symbol (lib_id "Device:C_Small") (at 195.58 77.47 270) (unit 1)
-    (in_bom yes) (on_board yes) (fields_autoplaced)
-    (property "Reference" "C305" (id 0) (at 195.5736 72.2081 90))
-    (property "Value" "1uF" (id 1) (at 195.5736 74.745 90))
-    (property "Footprint" "" (id 2) (at 195.58 77.47 0)
-      (effects (font (size 1.27 1.27)) hide)
-    )
-    (property "Datasheet" "~" (id 3) (at 195.58 77.47 0)
+  (symbol (lib_id "Device:C_Small") (at 193.04 74.93 180) (unit 1)
+    (in_bom yes) (on_board yes) (fields_autoplaced)
+    (property "Reference" "C305" (id 0) (at 195.3641 74.0889 0)
+      (effects (font (size 1.27 1.27)) (justify right))
+    )
+    (property "Value" "1uF" (id 1) (at 195.3641 76.6258 0)
+      (effects (font (size 1.27 1.27)) (justify right))
+    )
+    (property "Footprint" "" (id 2) (at 193.04 74.93 0)
+      (effects (font (size 1.27 1.27)) hide)
+    )
+    (property "Datasheet" "~" (id 3) (at 193.04 74.93 0)
       (effects (font (size 1.27 1.27)) hide)
     )
@@
       (effects (font (size 1.27 1.27)) hide)
     )
+    (pin "1")
+  )
+  (symbol (lib_id "power:GND") (at 193.04 85.09 0) (unit 1)
+    (in_bom yes) (on_board yes) (fields_autoplaced)
+    (property "Reference" "#PWR0304" (id 0) (at 193.04 91.44 0)
+      (effects (font (size 1.27 1.27)) hide)
+    )
+    (property "Value" "GND" (id 1) (at 193.04 89.5334 0))
+    (property "Footprint" "" (id 2) (at 193.04 85.09 0)
+      (effects (font (size 1.27 1.27)) hide)
+    )
+    (property "Datasheet" "" (id 3) (at 193.04 85.09 0)
+      (effects (font (size 1.27 1.27)) hide)
+    )
