File: KiCad/SignalSnagger/antenna_diagram.kicad_sch (KiCad schematic)
At the start: 0 parts

Commit message: Rev 0.28
Adding footprints to schematic: ~10% done
Other:
- note added: "Note for reference only and use the pins #'s in the root page of the schematic. Reason pin 7 and 8 were swapped: to get proper phasing of this sense loop."
Changed lines of the file:
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@@
     )
   )
+  (text "Note for reference only and use\nthe pins #'s in the root page of\nthe schematic. Reason pin  7 and 8\nwere swapped: to get proper \nphasing of this sense loop."
+    (at 81.28 152.4 0)
+    (effects (font (size 1.27 1.27)) (justify left bottom))
+  )
 )
