File: KiCad/SignalSnagger/SignalSnagger.kicad_pcb (KiCad board)
At the start: 4 copper layers, 133.4 x 44.3 mm, 212 parts, among them J102 69830-008LF, J104 69830-008LF, J105 36-5005-ND, J106 36-5006-ND, J107 36-5006-ND, J108 36-5005-ND, J203 Conn_01x02, J204 Conn_01x02, J208 Conn_01x04, J209 Conn_01x04, J218 Conn_01x02, J219 Conn_01x02, J301 35RASMT2BHSNTRX, J302 36-5005-ND, J304 36-5006-ND, J903 36-5005-ND, P201 ISP/PDI, Q101 MMBT2222A, Q102 MMBT2222A, Q103 MMBT2222A, Q201 NTS4173PT1G, Q202 BSS138W-7-F, SW201 SW_SPST, SW202 SW_SPST, SW203 PEC12R-4225F-S0024, T101 Coilcraft_PWB-4-CLC, T901 Coilcraft_PWB-4-CLC, U101 MIC6211, U102 QS3253QG8, U103 REF4132B33, U104 DG9422E, U105 DG9422E, U106 MCP4726, U201 AVR128DA48, U202 SI5351, U203 LP2985-5.0, U204 LP2985-3.3, U205 EA_DOGS104W-A, U206 LP2985-3.3, U302 TS912IDT, U303 MCP4018T-503E, U304 LM386, U901 TS912IDT, U902 LM386, U903 MCP4018T-503E, X202 25 MHz, X901 ECS-327TXO-30-TR

Commit message: Schematic & PCB Updates
o JFET sense amp option
o U301
Note: PCB changes are incomplete
Parts:
- added C109: 1nF, Capacitor_SMD:C_0603_1608Metric, F.Cu at (106.0, 85.5)
- added C302: 100nF, Capacitor_SMD:C_0603_1608Metric, F.Cu at (155.2, 99.8)
- added C304: 3.3nF, Capacitor_SMD:C_0603_1608Metric, F.Cu at (151.6, 101.4)
- added JP101: Jumper_2_Bridged, Jumper:Jumper_THT-1x02_Bridged_Circular, B.Cu at (89.6, 82.2)
- added JP102: Jumper_2_Bridged, Jumper:Jumper_THT-1x02_Bridged_Circular, B.Cu at (89.4, 110.2)
- added Q104: MBFJ310, Package_TO_SOT_SMD:SOT-23, F.Cu at (103.4, 83.8)
- added R114: 1k, Resistor_SMD:R_0603_1608Metric, F.Cu at (104.4, 87.3)
- added R315: 10, Resistor_SMD:R_0603_1608Metric, F.Cu at (201.4, 93.5)
- added U301: DG9422E, Package_SO:TSOP-6_1.65x3.05mm_P0.95mm, F.Cu at (155.2, 102.5)
- C116, C919: value 390pF -> 1000pF
- JP103, JP107: value Jumper_2_Bridged -> Jumper_2_Open; footprint Jumper:Jumper_THT-1x02_Bridged_Circular -> Jumper:Jumper_THT-1x02_Open_Circular
- R113, R915: value 4.99k -> 10k
- moved J302 28.9 mm to (139.7, 125.9)
- moved J903 22.7 mm to (147.2, 126.4)
- moved JP107 2.01 mm to (86.9, 110.2)
- moved JP103 1.79 mm to (87.0, 82.2)
- moved JP202 0.06 mm to (131.3, 79.4)
Connections:
- net ASSI_FAR renamed /Processor/ADC5
- C311 pad 1: Net-(C309-Pad1) -> Net-(U302B-OUT)
- C313 pad 1: Net-(C309-Pad1) -> Net-(U302B-OUT)
- C325 pad 1: Headphone -> Net-(JP301-A)
- C919 pad 1: Net-(C919-Pad1) -> Net-(U901A-OUT)
- C919 pad 2: Net-(C919-Pad2) -> Net-(U901A--)
- C920 pad 1: Net-(C919-Pad2) -> Net-(U901A-OUT)
- J301 pad 4: Headphone -> Net-(JP301-A)
- JP301 pad 1: Headphone -> Net-(JP301-A)
- Q102 pad 3: Net-(C109-Pad2) -> Net-(Q102-C)
- R108 pad 2: Net-(R108-Pad2) -> Net-(T101-PB)
- R109 pad 2: Net-(R109-Pad2) -> Net-(T101-PA)
- R301 pad 1: Net-(C309-Pad1) -> Net-(U302B-OUT)
- R306 pad 2: Net-(C309-Pad1) -> Net-(U302B-OUT)
- R914 pad 1: Net-(C919-Pad1) -> Net-(U901A--)
- R915 pad 1: Net-(C919-Pad1) -> Net-(U901A-OUT)
- R915 pad 2: Net-(C919-Pad2) -> Net-(U901A--)
- R930 pad 1: Net-(C919-Pad2) -> Net-(U901A-OUT)
- T101 pad 1: Net-(R109-Pad2) -> Net-(T101-PA)
- T101 pad 3: Net-(R108-Pad2) -> Net-(T101-PB)
- T101 pad 6: Net-(C109-Pad2) -> Net-(Q102-C)
- U201 pad 9: /Processor/PB5 -> Analog_Audio_Out
- U302 pad 7: Net-(C309-Pad1) -> Net-(U302B-OUT)
- U901 pad 1: Net-(C919-Pad2) -> Net-(U901A-OUT)
- U901 pad 2: Net-(C919-Pad1) -> Net-(U901A--)
Routing:
- net (no net): track 0.00 -> 41.1 mm, vias 0 -> 3
- net Net-(C919-Pad2): track 29.4 -> 0.00 mm, vias 3 -> 0
- net GNDD: track 563.7 -> 590.8 mm, vias 135 -> 137
- net Net-(C309-Pad1): track 19.3 -> 1.63 mm
- net GND: track 831.3 -> 814.6 mm, vias 268 -> 266
- net Net-(Q102-C): track 0.00 -> 14.7 mm, vias 0 -> 1
- net +VSW: track 258.7 -> 272.3 mm
- net Net-(C109-Pad2): track 14.7 -> 2.14 mm, vias 1 -> 0
- net Net-(C919-Pad1): track 11.8 -> 0.00 mm
- net Net-(JP105-B): track 23.4 -> 34.8 mm, vias 1 -> 2
- net Net-(U302B-OUT): track 0.00 -> 11.0 mm
- net Net-(Q101-B): track 19.7 -> 28.5 mm
- net Net-(JP301-A): track 0.00 -> 7.35 mm
- net Net-(T101-PB): track 0.00 -> 6.77 mm, vias 0 -> 1
- net Net-(R108-Pad2): track 6.77 -> 0.00 mm, vias 1 -> 0
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